File: SkyForge Hardware/Design/SkyForge.kicad_sch (KiCad schematic)
At the start: 13 parts, among them J1 GY-521 MPU6050, J2 0.96" SSD1306 OLED, J3 PS2 Joystick, SW1 SW_Push, SW2 SW_Push, SW3 SW_Push, SW4 SW_Push, U1 ESP32-DEVKIT-V1

Commit message: added SkyForge Hardware KiCAD files
Other:
- title: SkyForge Controller -> SkyForge Controller SCH
Changed lines of the file:
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@@
 	(paper "A4")
 	(title_block
-		(title "SkyForge Controller")
+		(title "SkyForge Controller SCH")
+		(date "2026-09-04")
 	)
 	(junction
